File: hw/usb.sch (KiCad schematic (older format))
At the start: 16 parts

Commit message: Work in progress.
Mostly comments in schematic for MCU, but also progress in USB sheet
Parts:
- added FB?: BLM18AG601SN1D, digikey-footprints:0603, symbol dk_Ferrite-Beads-and-Chips:BLM18AG601SN1D
- added R? (x6): 10k, symbol Device:R_Small_US
- added R?: 100k, symbol Device:R_Small_US
- added R?: 649R, symbol Device:R_Small_US
- R? (x2): value R_Small_US -> 5k1
Connections:
- wire segments 55 -> 84
- no-connect marks 2 -> 4
Other:
- moved on the sheet: C?, F?, J?, R?, U?, Y?
